File: src/left/ergoV.kicad_pcb (KiCad board)
At the start: 2 copper layers, 133.4 x 86.2 mm, 63 parts, among them J1 USB_C_Receptacle_USB2.0_16P, Q1 AO3401A, SW1 SW_Push_3pin_GND, SW10 SW_Push_3pin_GND, SW11 SW_Push_3pin_GND, SW12 SW_Push_3pin_GND, SW13 SW_Push_3pin_GND, SW14 SW_Push_3pin_GND, SW15 SW_Push_3pin_GND, SW16 SW_Push_3pin_GND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

Commit message: Finished pcb, started working on readme
Parts:
- added H1: MountingHole, MountingHole:MountingHole_2.7mm_M2.5, F.Cu at (128.0, 114.3)
- added H2: MountingHole, MountingHole:MountingHole_2.7mm_M2.5, F.Cu at (142.3, 114.3)
Routing:
- net COL1: track 168.9 -> 169.8 mm

Commit message: Finished readme and updated the pcb
Parts:
- R1, R2: footprint Resistor_SMD:R_0603_1608Metric -> Resistor_SMD:R_0402_1005Metric
- moved BT1 89.9 mm to (107.3, 118.0)
Routing:
- net VBAT: track 27.0 -> 178.0 mm, vias 2 -> 6
- net ROW0: track 131.0 -> 132.6 mm
- net +5V: track 52.4 -> 51.0 mm
- net COL0: track 197.7 -> 197.2 mm
- net GND: vias 31 -> 30
