File: src/right/ergoVright.kicad_sch (KiCad schematic)
At the start: 63 parts, among them J1 USB_C_Receptacle_USB2.0_16P, Q1 AO3401A, SW1 SW_Push_3pin_GND, SW10 SW_Push_3pin_GND, SW11 SW_Push_3pin_GND, SW12 SW_Push_3pin_GND, SW13 SW_Push_3pin_GND, SW14 SW_Push_3pin_GND, SW15 SW_Push_3pin_GND, SW16 SW_Push_3pin_GND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

Commit message: Finished pcb, started working on readme
Parts:
- added H1, H2: MountingHole, MountingHole:MountingHole_2.7mm_M2.5, symbol Mechanical:MountingHole
Changed lines of the file:
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@@
+	)
+	(symbol
+		(lib_id "Mechanical:MountingHole")
+		(at 223.52 134.62 0)
+		(unit 1)
+		(exclude_from_sim no)
+		(in_bom no)
+		(on_board yes)
+		(dnp no)
+		(fields_autoplaced yes)
+		(property "Reference" "H2"
+			(at 226.06 133.3499 0)
+			(effects
+				(font
+					(size 1.27 1.27)
+				)
+				(justify left)
+			)
+		)
+		(property "Value" "MountingHole"
+			(at 226.06 135.8899 0)
+			(effects
+				(font
+					(size 1.27 1.27)
+				)
+				(justify left)
+			)
+		)
+		(property "Footprint" "MountingHole:MountingHole_2.7mm_M2.5"
+			(at 223.52 134.62 0)
+			(effects
+				(font
+					(size 1.27 1.27)
+				)
+				(hide yes)
+			)
+		)
+		(property "Datasheet" "~"
+			(at 223.52 134.62 0)
+			(effects
+				(font
+					(size 1.27 1.27)
+				)
+				(hide yes)
+			)
+		)
+		(property "Description" "Mounting Hole without connection"
+			(at 223.52 134.62 0)
+			(effects
+				(font
+					(size 1.27 1.27)
+				)
+				(hide yes)
+			)
+		)
+		(instances
+			(project "ergoVright"
+				(path "/beacc4b6-f585-426a-9d0b-4a4efbedcb24"
+					(reference "H2")
+					(unit 1)
+				)
+			)
+		)
 	)
 	(symbol
@@
 					(unit 1)
 				)
+			)
+		)
+	)
+	(symbol
+		(lib_id "Mechanical:MountingHole")
+		(at 200.66 134.62 0)
+		(unit 1)
+		(exclude_from_sim no)
+		(in_bom no)
+		(on_board yes)
+		(dnp no)
+		(fields_autoplaced yes)
+		(property "Reference" "H1"
+			(at 203.2 133.3499 0)
+			(effects
+				(font
+					(size 1.27 1.27)
+				)
+				(justify left)
+			)
+		)
+		(property "Value" "MountingHole"
+			(at 203.2 135.8899 0)
+			(effects
+				(font
+					(size 1.27 1.27)
+				)
+				(justify left)
+			)
+		)
+		(property "Footprint" "MountingHole:MountingHole_2.7mm_M2.5"
+			(at 200.66 134.62 0)
+			(effects
+				(font
+					(size 1.27 1.27)
+				)
+				(hide yes)
+			)
+		)
+		(property "Datasheet" "~"
+			(at 200.66 134.62 0)
+			(effects
+				(font
+					(size 1.27 1.27)
+				)
+				(hide yes)
+			)
+		)
+		(property "Description" "Mounting Hole without connection"
+			(at 200.66 134.62 0)
+			(effects
+				(font
+					(size 1.27 1.27)
+				)
+				(hide yes)
+			)
+		)
+		(instances
+			(project "ergoVright"
+				(path "/beacc4b6-f585-426a-9d0b-4a4efbedcb24"
+					(reference "H1")
+					(unit 1)
+				)

Commit message: Finished readme and updated the pcb
Parts:
- BT1: LCSC C265016 -> (none)
- C1, C22: LCSC C23687 -> C19666
- C11, C2, C3, C4: LCSC C15525 -> C19702
- R1, R2: footprint Resistor_SMD:R_0603_1608Metric -> Resistor_SMD:R_0402_1005Metric; LCSC C11896 -> C25100
- R11: LCSC C4109 -> C22975
- R12: LCSC C25117 -> C23179
- R3, R4: LCSC C25905 -> C23186
- R7: LCSC C25744 -> C25804
- U1: LCSC (none) -> C14879
- U2: LCSC C14879 -> C5180249
- U4: LCSC C5180249 -> C67380
Changed lines of the file:
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@@
 			)
 		)
-		(property "LCSC" "C265016"
+		(property "LCSC" ""
 			(at 107.95 165.1 0)
 			(effects
@@
 			)
 		)
-		(property "LCSC" "C25905"
+		(property "LCSC" "C23186"
 			(at 57.15 148.59 90)
 			(effects
@@
 			)
 		)
-		(property "LCSC" "C15525"
+		(property "LCSC" "C19702"
 			(at 91.44 182.88 0)
 			(effects
@@
 			)
 		)
-		(property "LCSC" "C25744"
+		(property "LCSC" "C25804"
 			(at 81.28 182.88 0)
 			(effects
@@
 			)
 		)
-		(property "LCSC" "C14879"
+		(property "LCSC" "C5180249"
 			(at 132.08 167.64 0)
 			(effects
@@
 			)
 		)
-		(property "Footprint" "Resistor_SMD:R_0603_1608Metric"
+		(property "Footprint" "Resistor_SMD:R_0402_1005Metric"
 			(at 60.96 93.218 90)
 			(effects
@@
 			)
 		)
-		(property "LCSC" "C11896"
+		(property "LCSC" "C25100"
 			(at 60.96 91.44 90)
 			(effects
@@
 			)
 		)
+		(property "LCSC" "C14879"
+			(at 109.22 88.9 0)
+			(effects
+				(font
+					(size 1.27 1.27)
+				)
+				(hide yes)
+			)
+		)
 		(pin "51"
 		)
@@
 			)
 		)
-		(property "LCSC" "C4109"
+		(property "LCSC" "C22975"
 			(at 116.84 173.99 0)
 			(effects
@@
 			)
 		)
-		(property "LCSC" "C5180249"
+		(property "LCSC" "C67380"
 			(at 55.88 115.57 0)
 			(effects
@@
 			)
 		)
-		(property "LCSC" "C15525"
+		(property "LCSC" "C19702"
 			(at 102.87 36.83 0)
 			(effects
@@
 			)
 		)
-		(property "LCSC" "C23687"
+		(property "LCSC" "C19666 "
 			(at 148.59 168.91 0)
 			(effects
@@
 			)
 		)
-		(property "Footprint" "Resistor_SMD:R_0603_1608Metric"
+		(property "Footprint" "Resistor_SMD:R_0402_1005Metric"
 			(at 60.96 90.678 90)
 			(effects
@@
 			)
 		)
-		(property "LCSC" "C11896"
+		(property "LCSC" "C25100"
 			(at 60.96 88.9 90)
 			(effects
@@
 			)
 		)
-		(property "LCSC" "C25905"
+		(property "LCSC" "C23186"
 			(at 57.15 151.13 90)
 			(effects
@@
 			)
 		)
-		(property "LCSC" "C25117"
+		(property "LCSC" "C23179"
 			(at 142.24 179.07 0)
 			(effects
@@
 			)
 		)
-		(property "LCSC" "C23687"
+		(property "LCSC" "C19666 "
 			(at 120.65 160.02 0)
 			(effects
@@
 			)
 		)
-		(property "LCSC" "C15525"
+		(property "LCSC" "C19702"
 			(at 97.79 26.67 0)
 			(effects
@@
 			)
 		)
-		(property "LCSC" "C15525"
+		(property "LCSC" "C19702"
 			(at 86.36 26.67 0)
 			(effects
